Commit message: Add files via upload

File: rover_simulation/urdf/jackal.urdf.xacro (robot description, xacro)
@@ -218,4 +218,30 @@
     <origin xyz="${mount_spacing} 0 0" />
   </joint>
+   <joint name="hokuyo_joint" type="fixed">
+    <axis xyz="0 1 0" />
+    <origin xyz="0 0 ${chassis_height}" rpy="0 0 0"/>
+    <parent link="chassis_link"/>
+    <child link="hokuyo_link"/>
+  </joint>
+  <!-- Hokuyo Laser -->
+  <link name="hokuyo_link">
+    <collision>
+      <origin xyz="0 0 0" rpy="0 0 0"/>
+      <geometry>
+    <box size="0.1 0.1 0.1"/>
+      </geometry>
+    </collision>
+    <visual>
+      <origin xyz="0 0 0" rpy="0 0 0"/>
+      <geometry>
+        <mesh filename="package://gujju/meshes/hokuyo.dae"/>
+      </geometry>
+    </visual>
+    <inertial>
+      <mass value="1e-5" />
+      <origin xyz="0 0 0" rpy="0 0 0"/>
+      <inertia ixx="1e-6" ixy="0" ixz="0" iyy="1e-6" iyz="0" izz="1e-6" />
+    </inertial>
+  </link>
   <!-- Bring in simulation data for Gazebo. -->
   <xacro:include filename="$(find gujju)/urdf/jackal.gazebo" />

Commit message: Add files via upload

File: rover_simulation/urdf/jackal.urdf.xacro (robot description, xacro)
@@ -22,5 +22,5 @@
         <origin xyz="0 0 0" rpy="${PI/2} 0 0"/>
         <geometry>
-          <mesh filename="package://jackal_description/meshes/jackal-wheel.stl"/>
+          <mesh filename="$(find robofest_rover)/meshes/jackal-wheel.stl"/>
         </geometry>
         <material name="black" />
@@ -90,5 +90,5 @@
       <origin xyz="0 0 ${footprint_vertical_offset}" rpy="${PI/2} 0 ${PI/2}"/>
       <geometry>
-        <mesh filename="package://jackal_description/meshes/jackal-base.stl"/>
+        <mesh filename="$(find robofest_rover)/meshes/jackal-base.stl"/>
       </geometry>
       <material name="dark_grey" />
@@ -115,5 +115,5 @@
       <visual>
         <geometry>
-          <mesh filename="package://jackal_description/meshes/jackal-fender.stl"/>
+          <mesh filename="$(find robofest_rover)/meshes/jackal-fender.stl"/>
         </geometry>
         <material name="yellow" />
@@ -125,5 +125,5 @@
       <visual>
         <geometry>
-          <mesh filename="package://jackal_description/meshes/accessory_fender.stl"/>
+          <mesh filename="$(find robofest_rover)/meshes/accessory_fender.stl"/>
         </geometry>
         <material name="yellow" />
@@ -146,5 +146,5 @@
       <visual>
         <geometry>
-          <mesh filename="package://jackal_description/meshes/jackal-fender.stl"/>
+          <mesh filename="$(find robofest_rover)/meshes/jackal-fender.stl"/>
         </geometry>
         <material name="yellow" />
@@ -156,5 +156,5 @@
       <visual>
         <geometry>
-          <mesh filename="package://jackal_description/meshes/accessory_fender.stl"/>
+          <mesh filename="$(find robofest_rover)/meshes/accessory_fender.stl"/>
         </geometry>
         <material name="yellow" />
@@ -218,16 +218,17 @@
     <origin xyz="${mount_spacing} 0 0" />
   </joint>
-   <joint name="hokuyo_joint" type="fixed">
+   <joint name="lidar_joint" type="fixed">
     <axis xyz="0 1 0" />
-    <origin xyz="0 0 ${chassis_height}" rpy="0 0 0"/>
+    <origin xyz="0 0 ${chassis_height+0.012}" rpy="0 0 0"/>
     <parent link="chassis_link"/>
-    <child link="hokuyo_link"/>
+    <child link="lidar"/>
   </joint>
   <!-- Hokuyo Laser -->
-  <link name="hokuyo_link">
+  <link name="lidar">
     <collision>
       <origin xyz="0 0 0" rpy="0 0 0"/>
       <geometry>
-    <box size="0.1 0.1 0.1"/>
+    <mesh
+          filename="$(find robofest_rover)/meshes/lidar.STL" />
       </geometry>
     </collision>
@@ -235,5 +236,6 @@
       <origin xyz="0 0 0" rpy="0 0 0"/>
       <geometry>
-        <mesh filename="package://gujju/meshes/hokuyo.dae"/>
+        <mesh
+          filename="$(find robofest_rover)/meshes/lidar.STL" />
       </geometry>
     </visual>
@@ -245,4 +247,4 @@
   </link>
   <!-- Bring in simulation data for Gazebo. -->
-  <xacro:include filename="$(find gujju)/urdf/jackal.gazebo" />
+  <xacro:include filename="$(find robofest_rover)/urdf/jackal.gazebo" />
 </robot>

Commit message: Add files via upload

File: rover_simulation/urdf/jackal.urdf.xacro (robot description, xacro)
@@ -22,5 +22,5 @@
         <origin xyz="0 0 0" rpy="${PI/2} 0 0"/>
         <geometry>
-          <mesh filename="package://jackal_description/meshes/jackal-wheel.stl"/>
+          <mesh filename="$(find robofest_rover)/meshes/jackal-wheel.stl"/>
         </geometry>
         <material name="black" />
@@ -90,5 +90,5 @@
       <origin xyz="0 0 ${footprint_vertical_offset}" rpy="${PI/2} 0 ${PI/2}"/>
       <geometry>
-        <mesh filename="package://jackal_description/meshes/jackal-base.stl"/>
+        <mesh filename="$(find robofest_rover)/meshes/jackal-base.stl"/>
       </geometry>
       <material name="dark_grey" />
@@ -115,5 +115,5 @@
       <visual>
         <geometry>
-          <mesh filename="package://jackal_description/meshes/jackal-fender.stl"/>
+          <mesh filename="$(find robofest_rover)/meshes/jackal-fender.stl"/>
         </geometry>
         <material name="yellow" />
@@ -125,5 +125,5 @@
       <visual>
         <geometry>
-          <mesh filename="package://jackal_description/meshes/accessory_fender.stl"/>
+          <mesh filename="$(find robofest_rover)/meshes/accessory_fender.stl"/>
         </geometry>
         <material name="yellow" />
@@ -146,5 +146,5 @@
       <visual>
         <geometry>
-          <mesh filename="package://jackal_description/meshes/jackal-fender.stl"/>
+          <mesh filename="$(find robofest_rover)/meshes/jackal-fender.stl"/>
         </geometry>
         <material name="yellow" />
@@ -156,5 +156,5 @@
       <visual>
         <geometry>
-          <mesh filename="package://jackal_description/meshes/accessory_fender.stl"/>
+          <mesh filename="$(find robofest_rover)/meshes/accessory_fender.stl"/>
         </geometry>
         <material name="yellow" />

Commit message: updated repo

File: rover_simulation/urdf/jackal.urdf.xacro (robot description, xacro)
@@ -22,5 +22,5 @@
         <origin xyz="0 0 0" rpy="${PI/2} 0 0"/>
         <geometry>
-          <mesh filename="$(find robofest_rover)/meshes/jackal-wheel.stl"/>
+          <mesh filename="$(find rover_simulation)/meshes/jackal-wheel.stl"/>
         </geometry>
         <material name="black" />
@@ -90,5 +90,5 @@
       <origin xyz="0 0 ${footprint_vertical_offset}" rpy="${PI/2} 0 ${PI/2}"/>
       <geometry>
-        <mesh filename="$(find robofest_rover)/meshes/jackal-base.stl"/>
+        <mesh filename="$(find rover_simulation)/meshes/jackal-base.stl"/>
       </geometry>
       <material name="dark_grey" />
@@ -115,5 +115,5 @@
       <visual>
         <geometry>
-          <mesh filename="$(find robofest_rover)/meshes/jackal-fender.stl"/>
+          <mesh filename="$(find rover_simulation)/meshes/jackal-fender.stl"/>
         </geometry>
         <material name="yellow" />
@@ -125,5 +125,5 @@
       <visual>
         <geometry>
-          <mesh filename="$(find robofest_rover)/meshes/accessory_fender.stl"/>
+          <mesh filename="$(find rover_simulation)/meshes/accessory_fender.stl"/>
         </geometry>
         <material name="yellow" />
@@ -146,5 +146,5 @@
       <visual>
         <geometry>
-          <mesh filename="$(find robofest_rover)/meshes/jackal-fender.stl"/>
+          <mesh filename="$(find rover_simulation)/meshes/jackal-fender.stl"/>
         </geometry>
         <material name="yellow" />
@@ -156,5 +156,5 @@
       <visual>
         <geometry>
-          <mesh filename="$(find robofest_rover)/meshes/accessory_fender.stl"/>
+          <mesh filename="$(find rover_simulation)/meshes/accessory_fender.stl"/>
         </geometry>
         <material name="yellow" />
@@ -230,5 +230,5 @@
       <geometry>
     <mesh
-          filename="$(find robofest_rover)/meshes/lidar.STL" />
+          filename="$(find rover_simulation)/meshes/lidar.STL" />
       </geometry>
     </collision>
@@ -237,5 +237,5 @@
       <geometry>
         <mesh
-          filename="$(find robofest_rover)/meshes/lidar.STL" />
+          filename="$(find rover_simulation)/meshes/lidar.STL" />
       </geometry>
     </visual>
@@ -247,4 +247,4 @@
   </link>
   <!-- Bring in simulation data for Gazebo. -->
-  <xacro:include filename="$(find robofest_rover)/urdf/jackal.gazebo" />
+  <xacro:include filename="$(find rover_simulation)/urdf/jackal.gazebo" />
 </robot>

Commit message: updated urdf

File: rover_simulation/urdf/jackal.urdf.xacro (robot description, xacro)
@@ -22,5 +22,5 @@
         <origin xyz="0 0 0" rpy="${PI/2} 0 0"/>
         <geometry>
-          <mesh filename="$(find rover_simulation)/meshes/jackal-wheel.stl"/>
+          <mesh filename="package://rover_simulation/meshes/jackal-wheel.stl"/>
         </geometry>
         <material name="black" />
@@ -90,5 +90,5 @@
       <origin xyz="0 0 ${footprint_vertical_offset}" rpy="${PI/2} 0 ${PI/2}"/>
       <geometry>
-        <mesh filename="$(find rover_simulation)/meshes/jackal-base.stl"/>
+        <mesh filename="package://rover_simulation/meshes/jackal-base.stl"/>
       </geometry>
       <material name="dark_grey" />
@@ -115,5 +115,5 @@
       <visual>
         <geometry>
-          <mesh filename="$(find rover_simulation)/meshes/jackal-fender.stl"/>
+          <mesh filename="package://rover_simulation/meshes/jackal-fender.stl"/>
         </geometry>
         <material name="yellow" />
@@ -125,5 +125,5 @@
       <visual>
         <geometry>
-          <mesh filename="$(find rover_simulation)/meshes/accessory_fender.stl"/>
+          <mesh filename="package://rover_simulation/meshes/accessory_fender.stl"/>
         </geometry>
         <material name="yellow" />
@@ -146,5 +146,5 @@
       <visual>
         <geometry>
-          <mesh filename="$(find rover_simulation)/meshes/jackal-fender.stl"/>
+          <mesh filename="package://rover_simulation/meshes/jackal-fender.stl"/>
         </geometry>
         <material name="yellow" />
@@ -156,5 +156,5 @@
       <visual>
         <geometry>
-          <mesh filename="$(find rover_simulation)/meshes/accessory_fender.stl"/>
+          <mesh filename="package://rover_simulation/meshes/accessory_fender.stl"/>
         </geometry>
         <material name="yellow" />
@@ -230,5 +230,5 @@
       <geometry>
     <mesh
-          filename="$(find rover_simulation)/meshes/lidar.STL" />
+          filename="package://rover_simulation/meshes/lidar.STL" />
       </geometry>
     </collision>
@@ -237,5 +237,5 @@
       <geometry>
         <mesh
-          filename="$(find rover_simulation)/meshes/lidar.STL" />
+          filename="package://rover_simulation/meshes/lidar.STL" />
       </geometry>
     </visual>
