Commit message: Some bugs in navigation pipeline

File: rover_simulation/urdf/rover.urdf (robot description, URDF)
Before this commit: robot rover, 13 links, 12 joints
Links:
- link base_link: geometry collision mesh filename=package://rover_simulation/meshes/base_link.STL; visual mesh filename=package://rover_simulation/meshes/base_link.STL
- link gps_Link: geometry collision mesh filename=package://rover_simulation/meshes/gps_Link.STL; visual mesh filename=package://rover_simulation/meshes/gps_Link.STL
- link left_Link: geometry collision mesh filename=package://rover_simulation/meshes/left_Link.STL; visual mesh filename=package://rover_simulation/meshes/left_Link.STL
- link left_wheel_1_Link: geometry collision mesh filename=package://rover_simulation/meshes/left_wheel_1_Link.STL; visual mesh filename=package://rover_simulation/meshes/left_wheel_1_Link.STL
- link left_wheel_2_Link: geometry collision mesh filename=package://rover_simulation/meshes/left_wheel_2_Link.STL; visual mesh filename=package://rover_simulation/meshes/left_wheel_2_Link.STL
- link left_wheel_3_Link: geometry collision mesh filename=package://rover_simulation/meshes/left_wheel_3_Link.STL; visual mesh filename=package://rover_simulation/meshes/left_wheel_3_Link.STL
- link lidar_link: geometry collision mesh filename=package://rover_simulation/meshes/lidar_link.STL; visual mesh filename=package://rover_simulation/meshes/lidar_link.STL
- link main_left_Link: geometry collision mesh filename=package://rover_simulation/meshes/main_left_Link.STL; visual mesh filename=package://rover_simulation/meshes/main_left_Link.STL
- link main_right_Link: geometry collision mesh filename=package://rover_simulation/meshes/main_right_Link.STL; visual mesh filename=package://rover_simulation/meshes/main_right_Link.STL
- link right_Link: geometry collision mesh filename=package://rover_simulation/meshes/right_Link.STL; visual mesh filename=package://rover_simulation/meshes/right_Link.STL
- link right_wheel_1_Link: geometry collision mesh filename=package://rover_simulation/meshes/right_wheel_1_Link.STL; visual mesh filename=package://rover_simulation/meshes/right_wheel_1_Link.STL
- link right_wheel_2_Link: geometry collision mesh filename=package://rover_simulation/meshes/right_wheel_2_Link.STL; visual mesh filename=package://rover_simulation/meshes/right_wheel_2_Link.STL
- link right_wheel_3_Link: geometry collision mesh filename=package://rover_simulation/meshes/right_wheel_3_Link.STL; visual mesh filename=package://rover_simulation/meshes/right_wheel_3_Link.STL
